Commit message: fix: Change spawn pose to fix gazebo spawn error
The spawn pose of the robot result in parts of it being inside the
wall.

File: my_robot/urdf/my_robot.xacro (robot description, xacro)
@@ -9,5 +9,5 @@
   <xacro:property name="chassis_length" value=".5"/>
   <xacro:property name="chassis_width" value=".4"/>
-  <xacro:property name="chassis_height" value=".45"/>
+  <xacro:property name="chassis_height" value=".55"/>
   <xacro:property name="chassis_mass" value="5.0"/>
   <xacro:property name="wheel_length" value="0.1"/>
@@ -22,5 +22,5 @@
   <xacro:property name="camera_size" value="0.05 0.1 0.05"/>
   <xacro:property name="camera_x" value="${chassis_length / 2}"/>
-  <xacro:property name="lidar_z" value="${.1 + (chassis_height / 2)}"/>
+  <xacro:property name="lidar_z" value="${0.05 + (chassis_height / 2)}"/>
   <xacro:property name="diff_drive_wheel_spec">
     <wheelSeparation>${wheel_y * 2}"</wheelSeparation>

Commit message: feat: use a new world/map and tune AMCL

File: my_robot/urdf/my_robot.xacro (robot description, xacro)
@@ -22,5 +22,6 @@
   <xacro:property name="camera_size" value="0.05 0.1 0.05"/>
   <xacro:property name="camera_x" value="${chassis_length / 2}"/>
-  <xacro:property name="lidar_z" value="${0.05 + (chassis_height / 2)}"/>
+  <xacro:property name="lidar_z" value="${0.15 + (chassis_height / 2)}"/>
+  <xacro:property name="lidar_x" value="${(chassis_length / 2) - 0.05}"/>
   <xacro:property name="diff_drive_wheel_spec">
     <!-- This works on Melodic, but not Kinetic:
@@ -166,5 +167,5 @@
   </link>
   <joint type="fixed" name="hokuyo_joint">
-    <origin xyz="0 0 ${lidar_z}" rpy="0 0 0"/>
+    <origin xyz="${lidar_x} 0 ${lidar_z}" rpy="0 0 0"/>
     <child link="hokuyo"/>
     <parent link="chassis"/>
